File: hw/vb129_cannify_micro/cannify_micro.kicad_pcb (KiCad board)
At the start: 2 copper layers, 18 x 43.5 mm, 93 parts, among them J1 Conn_01x15, J2 Conn_01x15, J3 USB_C_Receptacle_USB2.0, J4 Pico-Lock 4P, J5 Pico-Lock 4P, U1 STM32G0B1KCTx, U2 LV14360SDDAR, U3 RT5760, U4 AOZ1376DI-02, U5 LMV358A, U6 74LVC1G08, U7 TS3A5223RSWR, U8 TCAN1044VDDF, X1 Osc 24MHz 50ppm 3.2x2.5mm

Commit message: Layout done.
Parts:
- removed C3, C4: 10nF, Capacitor_SMD:C_0402_1005Metric
- removed D13: Schottky 3A, vhrd_diode:D_SOD-123F
- removed JP1: Jumper board, Jumper:SolderJumper-2_P1.3mm_Open_RoundedPad1.0x1.5mm
- removed R26: 0, Resistor_SMD:R_0402_1005Metric
- removed R9: 100K, Resistor_SMD:R_0402_1005Metric
- removed the TP2 at (156.3, 53.7)
- removed TP3, TP4, TP7: TestPoint_Probe, TestPoint:TestPoint_Pad_D1.5mm
- removed X1: Osc 24MHz 50ppm 3.2x2.5mm, vhrd_crystal:Oscillator_SMD_Abracon_ASE-4Pin_3.2x2.5mm
- added C24: 100nF, Capacitor_SMD:C_0402_1005Metric, F.Cu at (151.8, 111.2)
- added C25: 4.7uF, Capacitor_SMD:C_0603_1608Metric, F.Cu at (153.2, 112.8)
- added C26: 1uF, Capacitor_SMD:C_0603_1608Metric, B.Cu at (144.4, 103.3)
- added C27: 100nF, Capacitor_SMD:C_0402_1005Metric, B.Cu at (147.5, 104.3)
- added C28: 1uF, Capacitor_SMD:C_0603_1608Metric, B.Cu at (144.4, 104.7)
- added C29: 12pF, Capacitor_SMD:C_0402_1005Metric, F.Cu at (146.0, 100.5)
- added C30: 12pF, Capacitor_SMD:C_0402_1005Metric, F.Cu at (146.0, 98.7)
- added C31: 24pF, Capacitor_SMD:C_0402_1005Metric, F.Cu at (142.8, 103.1)
- added D14: LED, LED_SMD:LED_0402_1005Metric, F.Cu at (154.0, 102.3)
- added FB1: MH1608-601Y, Inductor_SMD:L_0603_1608Metric, B.Cu at (149.6, 104.0)
- added JP2: Jumper (Short), Jumper:SolderJumper-2_P1.3mm_Bridged_RoundedPad1.0x1.5mm, F.Cu at (140.6, 107.4)
- added JP3: Jumper (Short), Jumper:SolderJumper-2_P1.3mm_Bridged_RoundedPad1.0x1.5mm, F.Cu at (154.1, 110.5)
- added R30: 39K2, Resistor_SMD:R_0402_1005Metric, B.Cu at (143.1, 110.2)
- added R31: 1K69, Resistor_SMD:R_0402_1005Metric, B.Cu at (144.1, 110.2)
- added Y1: 32.768kHz, vhrd_crystal:ECX-.327-CDX-1293, F.Cu at (148.8, 99.8)
- added Y2: 12MHz, Crystal:Crystal_SMD_3225-4Pin_3.2x2.5mm, F.Cu at (142.1, 100.4)
- C1, C19, C2, D4, D5: moved to B.Cu
- C20: value 10uF -> 4.7uF; footprint Capacitor_SMD:C_0805_2012Metric -> Capacitor_SMD:C_0603_1608Metric; moved to B.Cu
- C21: value 10nF -> 24pF
- C6, C7, D8, D9, R15, R16, R17, R22, R6, R7, R8: moved to F.Cu
- D1, D2, D3: value RCLAMP0502BA -> ESD
- D11: value Vbr=53V Vcl=77V -> Vbr=56V; footprint Diode_SMD:D_SOD-123F -> vhrd_diode:TVS_SOD-123F
- J1, J2: value Conn_01x15 -> Conn_01x20; footprint Connector_PinHeader_2.54mm:PinHeader_1x15_P2.54mm_Vertical -> Connector_PinHeader_2.54mm:PinHeader_1x20_P2.54mm_Vertical
- R27: value 10k -> 1K69
- R28: value 0 -> 10K; moved to B.Cu
- R3: value 4K7 -> 16K2; moved to B.Cu
- R4: value 10K -> 1K69; moved to B.Cu
- U1: value STM32G0B1KCTx -> STM32G0B1CETxN; footprint Package_QFP:LQFP-32_7x7mm_P0.8mm -> Package_QFP:LQFP-48_7x7mm_P0.5mm
- U2: footprint Package_SO:SOIC-8-1EP_3.9x4.9mm_P1.27mm_EP2.95x4.9mm_Mask2.71x3.4mm_ThermalVias -> vhrd_generic:SOIC-8-1EP_TI_NOVIA; moved to F.Cu
- moved R5 62.4 mm to (154.0, 119.8), turned to 90 degrees
- moved TP1 33.4 mm to (154.0, 88.6)
- moved R3 33.3 mm to (145.0, 110.2), turned to -90 degrees
- moved R4 32.1 mm to (146.0, 110.2), turned to 90 degrees
- moved TP5 26.5 mm to (154.0, 86.0)
- moved TP2 21.0 mm to (140.6, 88.6)
- moved C9 18.3 mm to (145.6, 124.8), turned to -90 degrees
- moved H2 16.0 mm to (141.6, 93.6)
- moved H1 16.0 mm to (153.0, 93.6)
- moved D5 15.8 mm to (147.4, 116.6)
- moved C23 15.7 mm to (153.5, 122.2), turned to 90 degrees
- moved C2 15.4 mm to (149.6, 86.6)
- moved U8 14.9 mm to (151.0, 121.0), turned to -90 degrees
- moved C5 13.9 mm to (149.0, 124.8), turned to -90 degrees
- moved R28 12.9 mm to (153.6, 97.5), turned to -90 degrees
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- renumbered TP6 to TP2
Connections:
- C16 pad 1: +VIN_USB_PR -> +5V0_DCDC
- C21 pad 1: +3V3_DCDC -> /HF_OSC_OUT
- C5 pad 1: /+5V0_DCDC_IN -> +VIN_CAN
- C6 pad 1: /+5V0_DCDC_IN -> +VIN_CAN
- D12 pad 1: /+5V0_DCDC_IN -> +VIN_CAN
- D12 pad 2: +VIN_CAN -> /+VCAN_F
- D3 pad 1: /USB_DN -> /USB_N
- D3 pad 2: /USB_DP -> /USB_P
- F1 pad 2: +VIN_CAN -> /+VCAN_F
- J1 pad 1: unconnected-(J1-Pin_1-Pad1) -> /PB4
- J1 pad 10: unconnected-(J1-Pin_10-Pad10) -> /VBAT
- J1 pad 11: unconnected-(J1-Pin_11-Pad11) -> /PA2
- J1 pad 12: unconnected-(J1-Pin_12-Pad12) -> /PA3
- J1 pad 13: unconnected-(J1-Pin_13-Pad13) -> /PA4
- J1 pad 14: unconnected-(J1-Pin_14-Pad14) -> /PA5
- J1 pad 15: unconnected-(J1-Pin_15-Pad15) -> +VIN_CAN
- J1 pad 2: unconnected-(J1-Pin_2-Pad2) -> /PB5
- J1 pad 3: unconnected-(J1-Pin_3-Pad3) -> /PB6
- J1 pad 4: unconnected-(J1-Pin_4-Pad4) -> /PB7
- J1 pad 5: unconnected-(J1-Pin_5-Pad5) -> /PB9
- J1 pad 6: unconnected-(J1-Pin_6-Pad6) -> /PF2_NRST
- J1 pad 7: unconnected-(J1-Pin_7-Pad7) -> GND
- J1 pad 8: unconnected-(J1-Pin_8-Pad8) -> /PA0
- J1 pad 9: unconnected-(J1-Pin_9-Pad9) -> /PA1
- J2 pad 1: unconnected-(J2-Pin_1-Pad1) -> /PB3
- J2 pad 10: unconnected-(J2-Pin_10-Pad10) -> /SWDIO
- J2 pad 11: unconnected-(J2-Pin_11-Pad11) -> +3V3_DCDC
- J2 pad 12: unconnected-(J2-Pin_12-Pad12) -> /+VDDIO2
- J2 pad 13: unconnected-(J2-Pin_13-Pad13) -> GND
- J2 pad 14: unconnected-(J2-Pin_14-Pad14) -> /PA9
- J2 pad 15: unconnected-(J2-Pin_15-Pad15) -> /PA8
- J2 pad 2: unconnected-(J2-Pin_2-Pad2) -> /PD3
- J2 pad 3: unconnected-(J2-Pin_3-Pad3) -> /PD2
- J2 pad 4: unconnected-(J2-Pin_4-Pad4) -> /PD0
- J2 pad 5: unconnected-(J2-Pin_5-Pad5) -> /PA15
- J2 pad 6: unconnected-(J2-Pin_6-Pad6) -> /PA10
- J2 pad 8: unconnected-(J2-Pin_8-Pad8) -> GND
- J2 pad 9: unconnected-(J2-Pin_9-Pad9) -> /SWCLK
- J3 pad A6: /USB_DP -> /USB_P
- J3 pad A7: /USB_DN -> /USB_N
- J3 pad B6: /USB_DP -> /USB_P
- J3 pad B7: /USB_DN -> /USB_N
- R14 pad 2: +VIN_USB_PR -> +5V0_DCDC
- R27 pad 2: +3V3_DCDC -> /LED
- R28 pad 1: /OSC_OUT -> GND
- R28 pad 2: /RCC_OSC_IN -> /SWCLK
- R3 pad 2: /USB_VBUS_DET -> /USB_VDIV
- R4 pad 1: /USB_VBUS_DET -> /USB_VDIV
- R6 pad 1: /+5V0_DCDC_IN -> +VIN_CAN
- TP1 pad 1: +VIN_USB -> /SWD_SEL
- TP2 pad 1: +VIN_USB_PR -> /VUSB_FLTB
- U1 pad 1: unconnected-(U1-PB9-Pad1) -> /CAN_STBY
- U1 pad 10: unconnected-(U1-PA3-Pad10) -> /PF2_NRST
- U1 pad 11: unconnected-(U1-PA4-Pad11) -> /PA0
- U1 pad 12: unconnected-(U1-PA5-Pad12) -> /PA1
- U1 pad 13: unconnected-(U1-PA6-Pad13) -> /PA2
- U1 pad 14: unconnected-(U1-PA7-Pad14) -> /PA3
- U1 pad 15: unconnected-(U1-PB0-Pad15) -> /PA4
- U1 pad 16: unconnected-(U1-PB1-Pad16) -> /PA5
- U1 pad 17: unconnected-(U1-PB2-Pad17) -> /PA6
- U1 pad 18: /CC1_PR -> /PA7
- U1 pad 19: /DBCC1 -> /PB0
- U1 pad 2: /RCC_OSC_IN -> /LF_OSC_IN
- U1 pad 20: unconnected-(U1-PC6-Pad20) -> /PB1
- U1 pad 21: unconnected-(U1-PA10/UCPD1_DBCC2-Pad21) -> /USB_VDIV
- U1 pad 22: unconnected-(U1-PA11/PA9-Pad22) -> /CAN_VDIV
- U1 pad 23: unconnected-(U1-PA12/PA10-Pad23) -> /PB11
- U1 pad 24: unconnected-(U1-PA13-Pad24) -> /PB12
- U1 pad 25: unconnected-(U1-PA14-Pad25) -> /PB13
- U1 pad 26: unconnected-(U1-PA15-Pad26) -> /LED
- U1 pad 27: unconnected-(U1-PB3-Pad27) -> /PB15
- U1 pad 28: unconnected-(U1-PB4-Pad28) -> /PA8
- U1 pad 29: unconnected-(U1-PB5-Pad29) -> /PA9
- U1 pad 3: unconnected-(U1-PC15-Pad3) -> /LF_OSC_OUT
- U1 pad 30: unconnected-(U1-PB6-Pad30) -> GND
- U1 pad 31: unconnected-(U1-PB7-Pad31) -> /+VDDIO2
- U1 pad 32: unconnected-(U1-PB8-Pad32) -> /PA10
- U1 pad 4: +3V3_DCDC -> /VBAT
- U1 pad 5: GND -> Net-(U1-VREF+)
- U1 pad 6: unconnected-(U1-PF2-Pad6) -> +3V3_DCDC
- U1 pad 7: unconnected-(U1-PA0-Pad7) -> GND
- U1 pad 8: unconnected-(U1-PA1-Pad8) -> /HF_OSC_IN
- U1 pad 9: unconnected-(U1-PA2-Pad9) -> /HF_OSC_OUT
- U2 pad 2: /+5V0_DCDC_IN -> +VIN_CAN
- U3 pad 6: /3V3_PG -> unconnected-(U3-PG-Pad6)
- U4 pad 1: +VIN_USB_PR -> +5V0_DCDC
- U4 pad 2: +VIN_USB_PR -> +5V0_DCDC
- U8 pad 1: /CAN_TXD -> /FDCAN_TX
- U8 pad 4: /CAN_RXD -> /FDCAN_RX
- U8 pad 8: /CAN_STB -> /CAN_STBY
Routing:
- net GND: track 0.00 -> 94.5 mm, vias 0 -> 58
- net +3V3_DCDC: track 0.00 -> 53.8 mm, vias 0 -> 11
- net +5V0_DCDC: track 0.00 -> 38.9 mm, vias 0 -> 15
- net /PB1: track 0.00 -> 35.9 mm, vias 0 -> 2
- net /SWD_SEL: track 0.00 -> 32.4 mm, vias 0 -> 4
- net /USB_N: track 0.00 -> 31.8 mm, vias 0 -> 2
- net /PB11: track 0.00 -> 31.3 mm, vias 0 -> 2
- net /USB_P: track 0.00 -> 30.4 mm, vias 0 -> 2
- net +VIN_USB: track 0.00 -> 28.8 mm, vias 0 -> 2
- net /PB0: track 0.00 -> 28.5 mm, vias 0 -> 1
- net /PA10: track 0.00 -> 28.3 mm, vias 0 -> 2
- net /PB4: track 0.00 -> 28.2 mm, vias 0 -> 1
- net /CAN_STBY: track 0.00 -> 26.9 mm, vias 0 -> 2
- net /PA7: track 0.00 -> 26.1 mm, vias 0 -> 1
- net /FDCAN_RX: track 0.00 -> 25.9 mm, vias 0 -> 2
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- added copper zone on B.Cu, net +3V3_DCDC
- added copper zone on In3.Cu, net +3V3_DCDC
- added copper zone on B.Cu, net +5V0_DCDC
- added copper zone on F.Cu, net +5V0_DCDC
- added copper zone on In3.Cu, net +5V0_DCDC
- added copper zone on B.Cu, net +VIN_CAN
- added copper zone on F.Cu, net +VIN_CAN
- added copper zone on B.Cu, net +VIN_USB
- added copper zone on B.Cu, net /+VCAN_F
- added copper zone on B.Cu, net /+VCAN_J
- added copper zone on F.Cu, net /+VCAN_J
- added copper zone on B.Cu, net /3V3_SW
- added copper zone on B.Cu, net /LV_SW
- added copper zone on F.Cu, net /LV_SW
- added copper zone on B.Cu, net GND
- added copper zone on F.Cu, net GND
- added copper zone on In1.Cu, net GND
- added copper zone on In4.Cu, net GND
Other:
- board size 18 x 43.5 mm -> 20.5 x 51 mm
- copper layers 2 -> 6
- board text added: "+"
- board text added: "CAN"
- board text added: "H"
- board text added: "IO2"
- board text added: "L"
- board text added: "TECH"
- board text added: "VBAT"
- board text added: "VHRD"
- board text added: "nify Micro"
